File: hardware/v0.1/zturn_breakout.kicad_pcb (KiCad board)
At the start: 2 copper layers, 13.3 x 20.8 mm, 2 parts, among them J2 Z-Turn JTAG, J4 HS3-JTAG

Commit message: Cleaned up v0.1 and began v1.0 schematic
Parts:
- removed J4: HS3-JTAG, Connector_PinHeader_2.00mm:PinHeader_2x07_P2.00mm_Horizontal
- added J2: HS3-JTAG, Connector_PinHeader_2.00mm:PinHeader_2x07_P2.00mm_Horizontal, B.Cu at (152.1, 105.0)
- renumbered J2 to J1
Changed lines of the file:
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@@
     (solder_mask_min_width 0.25)
     (aux_axis_origin 0 0)
-    (visible_elements FFFFFF7F)
+    (visible_elements 7FFFFFFF)
     (pcbplotparams
       (layerselection 0x010fc_ffffffff)
@@
   (net 7 /JTAG_TMS)
   (net 8 /VREF)
-  (net 9 "Net-(J4-Pad12)")
+  (net 9 "Net-(J1-Pad12)")
   (net_class Default "This is the default net class."
     (clearance 0.2)
@@
     (add_net /VREF)
     (add_net GND)
+    (add_net "Net-(J1-Pad12)")
     (add_net "Net-(J2-Pad12)")
-    (add_net "Net-(J4-Pad12)")
   )
   (module Connector_PinHeader_2.00mm:PinHeader_2x07_P2.00mm_Horizontal (layer B.Cu)
@@
     (descr "Through hole angled pin header, 2x07, 2.00mm pitch, 4.2mm pin length, double rows")
     (tags "Through hole angled pin header THT 2x07 2.00mm double row")
-    (fp_text reference J4 (at 2.032 2.032) (layer B.SilkS)
+    (fp_text reference J2 (at 2.794 2.413) (layer B.SilkS)
       (effects (font (size 1 1) (thickness 0.15)) (justify mirror))
     )
@@
       (net 1 GND))
     (pad 12 thru_hole oval (at 2 -10) (size 1.35 1.35) (drill 0.8) (layers *.Cu *.Mask)
-      (net 9 "Net-(J4-Pad12)"))
+      (net 3 "Net-(J2-Pad12)"))
     (pad 11 thru_hole oval (at 0 -10) (size 1.35 1.35) (drill 0.8) (layers *.Cu *.Mask)
       (net 1 GND))
@@
     (descr "Through hole straight socket strip, 2x07, 2.54mm pitch, double cols (from Kicad 4.0.7), script generated")
     (tags "Through hole socket strip THT 2x07 2.54mm double row")
-    (fp_text reference J2 (at 2.286 1.27) (layer B.SilkS)
+    (fp_text reference J1 (at 2.667 1.651) (layer B.SilkS)
       (effects (font (size 1 1) (thickness 0.15)) (justify mirror))
     )
@@
       (net 1 GND))
     (pad 12 thru_hole oval (at -2.54 -12.7) (size 1.7 1.7) (drill 1) (layers *.Cu *.Mask)
-      (net 3 "Net-(J2-Pad12)"))
+      (net 9 "Net-(J1-Pad12)"))
     (pad 11 thru_hole oval (at 0 -12.7) (size 1.7 1.7) (drill 1) (layers *.Cu *.Mask)
       (net 1 GND))
