File: hardware/v1.0/zturn_breakout_v1.0.sch (KiCad schematic (older format))
At the start: 3 parts

Commit message: Completed schematic and layout of v1.0
Parts:
- added J10: PMOD7, zturn_breakout:PinSocket_2x06_P2.54mm_Horizontal, symbol Connector_Generic:Conn_02x06_Top_Bottom
- added J11: PMOD8, zturn_breakout:PinSocket_2x06_P2.54mm_Horizontal, symbol Connector_Generic:Conn_02x06_Top_Bottom
- added J12: PMOD9, zturn_breakout:PinSocket_2x06_P2.54mm_Horizontal, symbol Connector_Generic:Conn_02x06_Top_Bottom
- added J13: PMOD10, zturn_breakout:PinSocket_2x06_P2.54mm_Horizontal, symbol Connector_Generic:Conn_02x06_Top_Bottom
- added J3: PMOD2, zturn_breakout:PinSocket_2x06_P2.54mm_Horizontal, symbol Connector_Generic:Conn_02x06_Top_Bottom
- added J4: PMOD3, zturn_breakout:PinSocket_2x06_P2.54mm_Horizontal, symbol Connector_Generic:Conn_02x06_Top_Bottom
- added J5: PMOD4, zturn_breakout:PinSocket_2x06_P2.54mm_Horizontal, symbol Connector_Generic:Conn_02x06_Top_Bottom
- added J6: PMOD5, zturn_breakout:PinSocket_2x06_P2.54mm_Horizontal, symbol Connector_Generic:Conn_02x06_Top_Bottom
- added J7: PMOD1, Connector_PinSocket_2.54mm:PinSocket_1x06_P2.54mm_Horizontal, symbol Connector_Generic:Conn_01x06
- added J9: PMOD6, zturn_breakout:PinSocket_2x06_P2.54mm_Horizontal, symbol Connector_Generic:Conn_02x06_Top_Bottom
- J1, J2: renamed from J?; footprint Connector_PinHeader_1.27mm:PinHeader_2x40_P1.27mm_Vertical -> Connector_PinHeader_1.27mm:PinHeader_2x40_P1.27mm_Vertical_SMD
- gave numbers to parts that had none: 1
Connections:
- net labels added: BP, HDMI_INT, IO_B13_LN12, IO_B13_LN13, IO_B13_LN14, IO_B13_LN15, IO_B13_LN21, IO_B13_LP12, IO_B13_LP13, IO_B13_LP14, IO_B13_LP15, IO_B13_LP21, IO_B35_LN1, IO_B35_LN10, IO_B35_LN11, IO_B35_LN12, IO_B35_LN13, IO_B35_LN14, IO_B35_LN15, IO_B35_LN16, IO_B35_LN17, IO_B35_LN18, IO_B35_LN19, IO_B35_LN2, IO_B35_LN20, IO_B35_LN21, IO_B35_LN22, IO_B35_LN23, IO_B35_LN24, IO_B35_LN3, IO_B35_LN4, IO_B35_LN5, IO_B35_LN6, IO_B35_LN7, IO_B35_LN8, IO_B35_LN9, IO_B35_LP1, IO_B35_LP10, IO_B35_LP11, IO_B35_LP12, IO_B35_LP13, IO_B35_LP14, IO_B35_LP15, IO_B35_LP16, IO_B35_LP17, IO_B35_LP18, IO_B35_LP19, IO_B35_LP2, IO_B35_LP20, IO_B35_LP21, IO_B35_LP22, IO_B35_LP23, IO_B35_LP24, IO_B35_LP3, IO_B35_LP4, IO_B35_LP5, IO_B35_LP6, IO_B35_LP7, IO_B35_LP8, IO_B35_LP9, LCD_DATA0, LCD_DATA1, LCD_DATA10, LCD_DATA11, LCD_DATA12, LCD_DATA13, LCD_DATA14, LCD_DATA15, LCD_DATA2, LCD_DATA3, LCD_DATA4, LCD_DATA5, LCD_DATA6, LCD_DATA7, LCD_DATA8, LCD_DATA9, LCD_DE, LCD_HSYNC, LCD_PCLK, LCD_VSYNC, MEMS_INTn, PS_MIO0, PS_MIO10, PS_MIO11, PS_MIO12, PS_MIO13, PS_MIO14, PS_MIO15, PS_MIO8, PS_MIO9, XADC_TEMP_N, XADC_TEMP_P, XADC_VCC, XDAC_INN0, XDAC_INP0
- net labels removed: IO_BP13_LN12, IO_BP13_LN13, IO_BP13_LN14, IO_BP13_LN15, IO_BP13_LN21, IO_BP13_LP12, IO_BP13_LP13, IO_BP13_LP14, IO_BP13_LP15, IO_BP13_LP21, JTAG_VREF, VDDIO_13_PL, VDDIO_34_PL, VDDIO_35_PL
- wire segments 146 -> 393
Other:
- note added: "1.8V from Z-Turn"
- note added: "JTAG_VREF"
- note added: "VDD18_KEY_BACKUP\n"
- note added: "VDDIO_13_PL\n"
- note added: "VDDIO_34_PL"
- note added: "VDDIO_35_PL"
- note added: "XADC_GND"
- moved on the sheet: J1, J2, J8
